File: pcb/probeInterfaceG2.kicad_pcb (KiCad board)
At the start: 2 copper layers, 123.2 x 75 mm, 211 parts, among them J1 Conn_02x07_Odd_Even, J2 Conn_02x01, J3 USB_B, J4 Debug, Q1 BCX56, Q10 BSS138, Q11 BSS138, Q12 BSS138, Q13 BSS138, Q14 BSS138, Q15 BSS138, Q2 BSS138, Q3 X0202NN, Q4 BSS138, Q5 BCX56, Q6 BSS138, Q7 BSS138, Q8 BSS138, Q9 BSS138, SW1 SW_Push, U1 NCP1117-3.3_SOT223, U10 HE3621A0500, U11 HE3621A0500, U12 HE3621A0500, U13 SN74AXC4T774RSVR, U14 HE3621A0500, U15 HE3621A0500, U16 HE3621A0500, U17 HE3621A0500, U18 SN74AXC4T774RSVR, U19 HE3621A0500, U2 W25Q128JVS, U20 HE3621A0500, U21 HE3621A0500, U22 HE3621A0500, U23 RP2040, U24 TBA 1-0511, U25 TBA 2-0511, U3 ADUM3160, U4 74HCT595, U5 74HCT595, U6 SN74AXC4T774RSVR, U7 MCP6002-xSN, U8 HE3621A0500, U9 74HCT595, Y2 12.000MHz 12p

Commit message: layout done
Parts:
- added C48: 10u, Capacitor_SMD:C_0805_2012Metric, F.Cu at (136.5, 87.3)
- moved C17 19.3 mm to (131.1, 126.1), turned to 180 degrees
- moved C15 15.3 mm to (133.0, 107.7)
- moved TP6 3.81 mm to (136.8, 102.6)
- moved R2 1.42 mm to (126.7, 121.6), turned to 90 degrees
- moved C16 1.27 mm to (131.8, 124.2)
- moved C21 0.90 mm to (147.6, 103.8)
- moved C20 0.64 mm to (146.4, 102.6)
- moved R36 0.64 mm to (119.0, 107.7)
- moved R77 0.64 mm to (123.5, 107.0)
- moved C12 0.63 mm to (138.7, 106.4)
- moved C14 0.63 mm to (144.4, 112.4)
- moved J2 0.63 mm to (114.0, 102.0)
- moved J3 0.63 mm to (100.9, 135.6)
- moved R34 0.63 mm to (119.0, 106.4)
- moved R78 0.63 mm to (123.5, 108.3)
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Routing:
- net +3V3: track 72.1 -> 289.1 mm, vias 12 -> 17
- net VBUS: track 278.3 -> 389.7 mm, vias 15 -> 19
- net +1V1: track 11.0 -> 24.0 mm, vias 4 -> 0
- net Net-(U4-QH'): track 0.00 -> 10.2 mm
- net /QSPI_SD0: track 23.2 -> 15.7 mm
- net VDD: track 243.5 -> 247.8 mm
- net /dacout: track 30.4 -> 26.1 mm, vias 0 -> 2
- net /QSPI_SCLK: track 17.0 -> 20.3 mm
- net /~{USB_BOOT}: track 34.8 -> 32.4 mm
- net /QSPI_SD3: track 21.3 -> 23.0 mm
- net /K9: track 109.3 -> 110.4 mm
- net /GPIO24: track 39.8 -> 38.9 mm
- net Net-(R22-Pad2): track 1.94 -> 2.83 mm
- net GND: track 156.1 -> 156.9 mm, vias 87 -> 88
- net /K7: track 117.7 -> 117.0 mm
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- added copper zone on F.Cu, net GND
- added copper zone on B.Cu, net VBUS
Other:
- board size 123.2 x 75 mm -> 122.8 x 75 mm
- board text added: "LTE probeInterfaceG2 M. Koch 06/2023"
- board text removed: "LTE probeInterfaceG2 M. Koch 2023"

Commit message: fixed drc
Parts:
- U23: footprint Package_DFN_QFN:QFN-56-1EP_7x7mm_P0.4mm_EP3.2x3.2mm_ThermalVias -> Package_DFN_QFN:QFN-56-1EP_7x7mm_P0.4mm_EP3.2x3.2mm
- moved C11 1.65 mm to (132.4, 118.5)
- moved TP2 1.27 mm to (119.7, 141.3)
- moved C13 0.89 mm to (138.6, 118.7)
- moved C12 0.64 mm to (138.7, 105.8)
- moved C16 0.64 mm to (131.8, 123.5)
- moved C17 0.63 mm to (131.1, 125.4)
Routing:
- net +3V3: track 289.1 -> 292.1 mm
- net VDD: track 247.8 -> 250.8 mm
- net /K2: track 74.4 -> 76.4 mm
- net Net-(J3-GND): track 79.5 -> 80.8 mm
- net Net-(U24-+Vin): track 41.5 -> 40.5 mm
- net /SWDIO: track 25.1 -> 25.8 mm
- net /GPIO23: track 14.8 -> 15.5 mm
- net /GPIO8: track 11.6 -> 12.3 mm
- net /K9: track 110.4 -> 111.0 mm
- net Net-(D5-A): track 43.0 -> 42.5 mm
- net GND: track 156.9 -> 157.4 mm, vias 88 -> 92

Commit message: reichelt bom added
Parts:
- D4: value LED -> LED gr
- D5: value LED -> LED rd
- R2, R3, R4: footprint Capacitor_SMD:C_0402_1005Metric -> Resistor_SMD:R_0402_1005Metric

Commit message: added digikey bom
Changed lines of the file:
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@@
       (plot_on_all_layers_selection 0x0000000_00000000)
       (disableapertmacros false)
-      (usegerberextensions false)
+      (usegerberextensions true)
       (usegerberattributes false)
       (usegerberadvancedattributes false)
@@
       (psa4output false)
       (plotreference true)
-      (plotvalue true)
+      (plotvalue false)
       (plotinvisibletext false)
       (sketchpadsonfab false)
-      (subtractmaskfromsilk false)
+      (subtractmaskfromsilk true)
       (outputformat 1)
       (mirror false)
@@
     (fp_line (start 13.28 20.34) (end 4.38 20.34)
       (stroke (width 0.1) (type solid)) (layer "F.Fab"))
-    (pad "1" thru_hole roundrect (at 0 0) (size 1.7 1.7) (drill 1) (layers "*.Cu" "*.Mask") (roundrect_rratio 0.147059)
+    (pad "1" thru_hole roundrect (at 0 0) (size 1.7 1.7) (drill 1) (layers "*.Cu" "*.Mask") (roundrect_rratio 0.1470588235)
       (net 1 "GND") (pinfunction "Pin_1") (pintype "passive"))
     (pad "2" thru_hole circle (at 2.54 0) (size 1.7 1.7) (drill 1) (layers "*.Cu" "*.Mask")
@@
     (fp_line (start 1 0.625) (end -1 0.625)
       (stroke (width 0.1) (type solid)) (layer "F.Fab"))
-    (pad "1" smd roundrect (at -0.9125 0 270) (size 1.025 1.4) (layers "F.Cu" "F.Paste" "F.Mask") (roundrect_rratio 0.243902)
+    (pad "1" smd roundrect (at -0.9125 0 270) (size 1.025 1.4) (layers "F.Cu" "F.Paste" "F.Mask") (roundrect_rratio 0.243902439)
       (net 93 "Net-(Q1-B)") (pintype "passive"))
-    (pad "2" smd roundrect (at 0.9125 0 270) (size 1.025 1.4) (layers "F.Cu" "F.Paste" "F.Mask") (roundrect_rratio 0.243902)
+    (pad "2" smd roundrect (at 0.9125 0 270) (size 1.025 1.4) (layers "F.Cu" "F.Paste" "F.Mask") (roundrect_rratio 0.243902439)
       (net 37 "VDD") (pintype "passive"))
     (model "${KICAD6_3DMODEL_DIR}/Resistor_SMD.3dshapes/R_0805_2012Metric.wrl"
@@
     (fp_line (start 3.5 3.5) (end -3.5 3.5)
       (stroke (width 0.1) (type solid)) (layer "F.Fab"))
-    (pad "" smd roundrect (at -0.8 -0.8 90) (size 1.29 1.29) (layers "F.Paste") (roundrect_rratio 0.193798))
-    (pad "" smd roundrect (at -0.8 0.8 90) (size 1.29 1.29) (layers "F.Paste") (roundrect_rratio 0.193798))
-    (pad "" smd roundrect (at 0.8 -0.8 90) (size 1.29 1.29) (layers "F.Paste") (roundrect_rratio 0.193798))
-    (pad "" smd roundrect (at 0.8 0.8 90) (size 1.29 1.29) (layers "F.Paste") (roundrect_rratio 0.193798))
+    (pad "" smd roundrect (at -0.8 -0.8 90) (size 1.29 1.29) (layers "F.Paste") (roundrect_rratio 0.1937976744))
+    (pad "" smd roundrect (at -0.8 0.8 90) (size 1.29 1.29) (layers "F.Paste") (roundrect_rratio 0.1937976744))
+    (pad "" smd roundrect (at 0.8 -0.8 90) (size 1.29 1.29) (layers "F.Paste") (roundrect_rratio 0.1937976744))
+    (pad "" smd roundrect (at 0.8 0.8 90) (size 1.29 1.29) (layers "F.Paste") (roundrect_rratio 0.1937976744))
     (pad "1" smd roundrect (at -3.4375 -2.6 90) (size 0.875 0.2) (layers "F.Cu" "F.Paste" "F.Mask") (roundrect_rratio 0.25)
       (net 5 "+3V3") (pinfunction "IOVDD") (pintype "power_in"))
