File: pcb/io.kicad_sch (KiCad schematic)
At the start: 7 parts, among them Q4 BSS138, U8 HE3621A0500

Commit message: reichelt bom added
Parts:
- C22: Reichelt (none) -> MUR GRM1555C1H10
- D1: Reichelt (none) -> 1N 4148WS DIO
- D3: Reichelt (none) -> BAT 54S DIO
- Q4: Reichelt (none) -> BSS 138 SMD
- R32: Reichelt (none) -> RND 0402 1 47
- R40: Reichelt (none) -> RND 155HP02 AC
- U8: Reichelt (none) -> LITT HE3621A0500
Changed lines of the file:
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@@
+      (effects (font (size 1.27 1.27)) hide)
+    )
+    (property "Reichelt" "MUR GRM1555C1H10" (at 123.19 95.25 0)
       (effects (font (size 1.27 1.27)) hide)
     )
@@
     )
     (property "Datasheet" "~" (at 149.86 92.71 0)
+      (effects (font (size 1.27 1.27)) hide)
+    )
+    (property "Reichelt" "RND 155HP02 AC" (at 149.86 92.71 0)
       (effects (font (size 1.27 1.27)) hide)
     )
@@
       (effects (font (size 1.27 1.27)) hide)
     )
+    (property "Reichelt" "RND 0402 1 47" (at 123.19 106.68 0)
+      (effects (font (size 1.27 1.27)) hide)
+    )
     (pin "1")
     (pin "2")
@@
       (effects (font (size 1.27 1.27)) hide)
     )
+    (property "Reichelt" "BAT 54S DIO" (at 100.33 123.19 0)
+      (effects (font (size 1.27 1.27)) hide)
+    )
     (pin "1")
     (pin "2")
@@
     )
     (property "Datasheet" "https://www.littelfuse.com/~/media/electronics/datasheets/reed_relays/littelfuse_reed_relays_he3600_datasheet.pdf.pdf" (at 168.91 71.12 0)
+      (effects (font (size 1.27 1.27)) hide)
+    )
+    (property "Reichelt" "LITT HE3621A0500" (at 168.91 71.12 0)
       (effects (font (size 1.27 1.27)) hide)
     )
@@
       (effects (font (size 1.27 1.27)) hide)
     )
+    (property "Reichelt" "1N 4148WS DIO" (at 143.51 71.12 0)
+      (effects (font (size 1.27 1.27)) hide)
+    )
     (pin "1")
     (pin "2")
@@
       (effects (font (size 1.27 1.27)) (justify left) hide)
     )
-    (pin "1")
+    (property "Reichelt" "BSS 138 SMD" (at 161.29 87.63 0)
+      (effects (font (size 1.27 1.27)) hide)
+    )
+    (pin "1")

Commit message: added digikey bom
Parts:
- C22: Digikey (none) -> 490-GCM1555C1H102GA16JDKR-ND
- D1: Digikey (none) -> 4878-1N4148WDKR-ND
- D3: Digikey (none) -> BAT54SLT1GOSDKR-ND
- Q4: Digikey (none) -> 1727-1143-1-ND
- R32: Digikey (none) -> 311-47.0LRCT-ND
- R40: Digikey (none) -> YAG3436CT-ND
- U8: Digikey (none) -> HE206-ND
Changed lines of the file:
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@@
+      (effects (font (size 1.27 1.27)) hide)
+    )
+    (property "Digikey" "490-GCM1555C1H102GA16JDKR-ND" (at 123.19 95.25 0)
       (effects (font (size 1.27 1.27)) hide)
     )
@@
     )
     (property "Reichelt" "RND 155HP02 AC" (at 149.86 92.71 0)
+      (effects (font (size 1.27 1.27)) hide)
+    )
+    (property "Digikey" "YAG3436CT-ND" (at 149.86 92.71 0)
       (effects (font (size 1.27 1.27)) hide)
     )
@@
       (effects (font (size 1.27 1.27)) hide)
     )
+    (property "Digikey" "311-47.0LRCT-ND" (at 123.19 106.68 0)
+      (effects (font (size 1.27 1.27)) hide)
+    )
     (pin "1")
     (pin "2")
@@
       (effects (font (size 1.27 1.27)) hide)
     )
+    (property "Digikey" "BAT54SLT1GOSDKR-ND" (at 100.33 123.19 0)
+      (effects (font (size 1.27 1.27)) hide)
+    )
     (pin "1")
     (pin "2")
@@
     )
     (property "Reichelt" "LITT HE3621A0500" (at 168.91 71.12 0)
+      (effects (font (size 1.27 1.27)) hide)
+    )
+    (property "Digikey" "HE206-ND" (at 168.91 71.12 0)
       (effects (font (size 1.27 1.27)) hide)
     )
@@
       (effects (font (size 1.27 1.27)) hide)
     )
+    (property "Digikey" "4878-1N4148WDKR-ND" (at 143.51 71.12 0)
+      (effects (font (size 1.27 1.27)) hide)
+    )
     (pin "1")
     (pin "2")
@@
       (effects (font (size 1.27 1.27)) hide)
     )
+    (property "Digikey" "1727-1143-1-ND" (at 161.29 87.63 0)
+      (effects (font (size 1.27 1.27)) hide)
+    )

Commit message: corrected digikey bom
Parts:
- C22: Digikey 490-GCM1555C1H102GA16JDKR-ND -> 490-GCM1555C1H102GA16JCT-ND
- D1: Digikey 4878-1N4148WDKR-ND -> 4878-1N4148WCT-ND
- D3: Digikey BAT54SLT1GOSDKR-ND -> BAT54SLT1GOSCT-ND
Changed lines of the file:
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@@
       (effects (font (size 1.27 1.27)) hide)
     )
-    (property "Digikey" "490-GCM1555C1H102GA16JDKR-ND" (at 123.19 95.25 0)
+    (property "Digikey" "490-GCM1555C1H102GA16JCT-ND" (at 123.19 95.25 0)
       (effects (font (size 1.27 1.27)) hide)
     )
@@
       (effects (font (size 1.27 1.27)) hide)
     )
-    (property "Digikey" "BAT54SLT1GOSDKR-ND" (at 100.33 123.19 0)
+    (property "Digikey" "BAT54SLT1GOSCT-ND" (at 100.33 123.19 0)
       (effects (font (size 1.27 1.27)) hide)
     )
@@
       (effects (font (size 1.27 1.27)) hide)
     )
-    (property "Digikey" "4878-1N4148WDKR-ND" (at 143.51 71.12 0)
-      (effects (font (size 1.27 1.27)) hide)
-    )
+    (property "Digikey" "4878-1N4148WCT-ND" (at 143.51 71.12 0)
+      (effects (font (size 1.27 1.27)) hide)
+    )
