File: pcb/probeInterfaceG2.kicad_sch (KiCad schematic)
At the start: 128 parts, among them J2 Conn_02x01, J3 USB_B, J4 Debug, Q1 BCX56, Q3 X0202NN, Q5 BCX56, SW1 SW_Push, U1 NCP1117-3.3_SOT223, U13 SN74AXC4T774RSVR, U18 SN74AXC4T774RSVR, U2 W25Q128JVS, U23 RP2040, U24 TBA 1-0511, U25 TBA 2-0511, U3 ADUM3160, U4 74HCT595, U5 74HCT595, U6 SN74AXC4T774RSVR, U7 MCP6002-xSN, U9 74HCT595, Y2 12.000MHz 12p

Commit message: corrected digikey bom
Parts:
- C19: Digikey 13-CC0402JPNPO9BN101DKR-ND -> 13-CC0402JPNPO9BN101CT-ND
- C2, C3: Digikey 13-CC0402JPNPO9BN180DKR-ND -> 311-1014-1-ND
- C27: Digikey 490-GCM1555C1H102GA16JDKR-ND -> 490-GCM1555C1H102GA16JCT-ND
- D2, D7: Digikey BAT54SLT1GOSDKR-ND -> BAT54SLT1GOSCT-ND
- D40: Digikey BZX84C3V6LT1GOSDKR-ND -> BZX84C3V6LT1GOSCT-ND
- F1: Digikey 0ZCJ0050FF2G -> 507-1802-1-ND
- R1, R5: Digikey 13-AC0402FR-131KLDKR-ND -> 13-AC0402FR-131KLCT-ND
- R30: Digikey 13-RC0402FR-1310RLDKR-ND -> 13-RC0402FR-1310RLCT-ND
- U1: Digikey AZ1117IH-3.3TRG1DIDKR-ND -> AZ1117IH-3.3TRG1DICT-ND
- U13, U18, U6: Digikey 296-SN74AXC4T774RSVRDKR-ND -> 296-SN74AXC4T774RSVRCT-ND
- U2: Digikey W25Q128JVSIQDKR-ND -> W25Q128JVSIQCT-ND
- U23: Digikey 2648-SC0914(13)DKR-ND -> 2648-SC0914(13)CT-ND
- U3: Digikey ADUM3160BRWZ-RLDKR-ND -> ADUM3160BRWZ-RLCT-ND
- Y2: Digikey ABM3B-12.000MHZ-12-N2Y-T -> 535-14827-1-ND
Changed lines of the file:
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@@
       (effects (font (size 1.27 1.27)) hide)
     )
-    (property "Digikey" "13-CC0402JPNPO9BN180DKR-ND" (at 35.56 163.83 0)
+    (property "Digikey" "311-1014-1-ND" (at 35.56 163.83 0)
       (effects (font (size 1.27 1.27)) hide)
     )
@@
       (effects (font (size 1.27 1.27)) hide)
     )
-    (property "Digikey" "13-CC0402JPNPO9BN180DKR-ND" (at 35.56 173.99 0)
+    (property "Digikey" "311-1014-1-ND" (at 35.56 173.99 0)
       (effects (font (size 1.27 1.27)) hide)
     )
@@
       (effects (font (size 1.27 1.27)) hide)
     )
-    (property "Digikey" "W25Q128JVSIQDKR-ND" (at 160.02 166.37 0)
+    (property "Digikey" "W25Q128JVSIQCT-ND" (at 160.02 166.37 0)
       (effects (font (size 1.27 1.27)) hide)
     )
@@
       (effects (font (size 1.27 1.27)) hide)
     )
-    (property "Digikey" "13-AC0402FR-131KLDKR-ND" (at 129.54 163.83 0)
+    (property "Digikey" "13-AC0402FR-131KLCT-ND" (at 129.54 163.83 0)
       (effects (font (size 1.27 1.27)) hide)
     )
@@
       (effects (font (size 1.27 1.27)) hide)
     )
-    (property "Digikey" "AZ1117IH-3.3TRG1DIDKR-ND" (at 193.04 34.29 0)
+    (property "Digikey" "AZ1117IH-3.3TRG1DICT-ND" (at 193.04 34.29 0)
       (effects (font (size 1.27 1.27)) hide)
     )
@@
       (effects (font (size 1.27 1.27)) hide)
     )
-    (property "Digikey" "13-AC0402FR-131KLDKR-ND" (at 68.58 173.99 0)
+    (property "Digikey" "13-AC0402FR-131KLCT-ND" (at 68.58 173.99 0)
       (effects (font (size 1.27 1.27)) hide)
     )
@@
       (effects (font (size 1.27 1.27)) hide)
     )
-    (property "Digikey" "BAT54SLT1GOSDKR-ND" (at 327.66 203.2 0)
+    (property "Digikey" "BAT54SLT1GOSCT-ND" (at 327.66 203.2 0)
       (effects (font (size 1.27 1.27)) hide)
     )
@@
       (effects (font (size 1.27 1.27)) hide)
     )
-    (property "Digikey" "13-CC0402JPNPO9BN101DKR-ND" (at 317.5 307.34 0)
+    (property "Digikey" "13-CC0402JPNPO9BN101CT-ND" (at 317.5 307.34 0)
       (effects (font (size 1.27 1.27)) hide)
     )
@@
       (effects (font (size 1.27 1.27)) hide)
     )
-    (property "Digikey" "296-SN74AXC4T774RSVRDKR-ND" (at 482.6 254 0)
+    (property "Digikey" "296-SN74AXC4T774RSVRCT-ND" (at 482.6 254 0)
       (effects (font (size 1.27 1.27)) hide)
     )
@@
       (effects (font (size 1.27 1.27)) hide)
     )
-    (property "Digikey" "296-SN74AXC4T774RSVRDKR-ND" (at 482.6 83.82 0)
+    (property "Digikey" "296-SN74AXC4T774RSVRCT-ND" (at 482.6 83.82 0)
       (effects (font (size 1.27 1.27)) hide)
     )
@@
       (effects (font (size 1.27 1.27)) hide)
     )
-    (property "Digikey" "490-GCM1555C1H102GA16JDKR-ND" (at 336.55 209.55 0)
+    (property "Digikey" "490-GCM1555C1H102GA16JCT-ND" (at 336.55 209.55 0)
       (effects (font (size 1.27 1.27)) hide)
     )
@@
       (effects (font (size 1.27 1.27)) hide)
     )
-    (property "Digikey" "2648-SC0914(13)DKR-ND" (at 317.5 118.11 0)
+    (property "Digikey" "2648-SC0914(13)CT-ND" (at 317.5 118.11 0)
       (effects (font (size 1.27 1.27)) hide)
     )
@@
       (effects (font (size 1.27 1.27)) hide)
     )
-    (property "Digikey" "296-SN74AXC4T774RSVRDKR-ND" (at 482.6 168.91 0)
+    (property "Digikey" "296-SN74AXC4T774RSVRCT-ND" (at 482.6 168.91 0)
       (effects (font (size 1.27 1.27)) hide)
     )
@@
       (effects (font (size 1.27 1.27)) hide)
     )
-    (property "Digikey" "ADUM3160BRWZ-RLDKR-ND" (at 109.22 95.25 0)
+    (property "Digikey" "ADUM3160BRWZ-RLCT-ND" (at 109.22 95.25 0)
       (effects (font (size 1.27 1.27)) hide)
     )
@@
       (effects (font (size 1.27 1.27)) hide)
     )
-    (property "Digikey" "BAT54SLT1GOSDKR-ND" (at 381 233.68 0)
+    (property "Digikey" "BAT54SLT1GOSCT-ND" (at 381 233.68 0)
       (effects (font (size 1.27 1.27)) hide)
     )
@@
       (effects (font (size 1.27 1.27)) hide)
     )
-    (property "Digikey" "0ZCJ0050FF2G" (at 138.43 34.29 90)
+    (property "Digikey" "507-1802-1-ND" (at 138.43 34.29 90)
       (effects (font (size 1.27 1.27)) hide)
     )
@@
       (effects (font (size 1.27 1.27)) hide)
     )
-    (property "Digikey" "13-RC0402FR-1310RLDKR-ND" (at 354.33 309.88 0)
+    (property "Digikey" "13-RC0402FR-1310RLCT-ND" (at 354.33 309.88 0)
       (effects (font (size 1.27 1.27)) hide)
     )
@@
       (effects (font (size 1.27 1.27)) hide)
     )
-    (property "Digikey" "ABM3B-12.000MHZ-12-N2Y-T" (at 50.8 168.91 90)
+    (property "Digikey" "535-14827-1-ND" (at 50.8 168.91 90)
       (effects (font (size 1.27 1.27)) hide)
     )
@@
       (effects (font (size 1.27 1.27)) hide)
     )
-    (property "Digikey" "BZX84C3V6LT1GOSDKR-ND" (at 375.92 322.58 0)
+    (property "Digikey" "BZX84C3V6LT1GOSCT-ND" (at 375.92 322.58 0)
       (effects (font (size 1.27 1.27)) hide)
     )
