File: pcb/probeInterfaceG2.kicad_sch (KiCad schematic)
At the start: 128 parts, among them J2 Conn_02x01, J3 USB_B, J4 Debug, Q1 BCX56, Q3 X0202NN, Q5 BCX56, SW1 SW_Push, U1 NCP1117-3.3_SOT223, U13 SN74AXC4T774RSVR, U18 SN74AXC4T774RSVR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

Commit message: PCB tested and firmware adapted, gpios and spi available, readme adapted, pcbSimple removed
Parts:
- R11, R13, R15, R17, R19, R21, R23, R25, R27, R29, R6, R7, R8: value 10k -> 20k
- R31: value 100R -> 68R
Other:
- note added: "470p on top"
- note added: "limiting circuit does not work very well"
Changed lines of the file:
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@@
     (effects (font (size 1.27 1.27)) (justify right bottom))
   )
+  (text "470p on top" (at 440.69 97.79 0)
+    (effects (font (size 1.27 1.27)) (justify left bottom))
+  )
   (text "Make sure C8 is close to pin 45 of RP2040" (at 257.81 59.69 0)
     (effects (font (size 1.27 1.27)) (justify left bottom))
@@
     (effects (font (size 1.27 1.27)) (justify left bottom))
   )
+  (text "limiting circuit does not work very well" (at 394.97 335.915 0)
+    (effects (font (size 1.27 1.27)) (justify left bottom))
+  )
   (text "14p for 12p crystal\n27p for 18p crystal" (at 19.05 156.21 0)
     (effects (font (size 1.27 1.27)) (justify left bottom))
@@
       (effects (font (size 1.27 1.27)) (justify left))
     )
-    (property "Value" "10k" (at 223.52 323.85 0)
+    (property "Value" "20k" (at 223.52 323.85 0)
       (effects (font (size 1.27 1.27)) (justify left))
     )
@@
       (effects (font (size 1.27 1.27)) (justify left))
     )
-    (property "Value" "10k" (at 198.12 323.85 0)
+    (property "Value" "20k" (at 198.12 323.85 0)
       (effects (font (size 1.27 1.27)) (justify left))
     )
@@
       (effects (font (size 1.27 1.27)) (justify left))
     )
-    (property "Value" "10k" (at 261.62 323.85 0)
+    (property "Value" "20k" (at 261.62 323.85 0)
       (effects (font (size 1.27 1.27)) (justify left))
     )
@@
       (effects (font (size 1.27 1.27)) (justify left))
     )
-    (property "Value" "10k" (at 134.62 323.85 0)
+    (property "Value" "20k" (at 134.62 323.85 0)
       (effects (font (size 1.27 1.27)) (justify left))
     )
@@
       (effects (font (size 1.27 1.27)) (justify left))
     )
-    (property "Value" "10k" (at 121.92 323.85 0)
+    (property "Value" "20k" (at 121.92 323.85 0)
       (effects (font (size 1.27 1.27)) (justify left))
     )
@@
       (effects (font (size 1.27 1.27)) (justify left))
     )
-    (property "Value" "10k" (at 160.02 323.85 0)
+    (property "Value" "20k" (at 160.02 323.85 0)
       (effects (font (size 1.27 1.27)) (justify left))
     )
@@
       (effects (font (size 1.27 1.27)) (justify left))
     )
-    (property "Value" "10k" (at 248.92 323.85 0)
+    (property "Value" "20k" (at 248.92 323.85 0)
       (effects (font (size 1.27 1.27)) (justify left))
     )
@@
       (effects (font (size 1.27 1.27)) (justify left))
     )
-    (property "Value" "100R" (at 378.46 335.28 0)
+    (property "Value" "68R" (at 378.46 335.28 0)
       (effects (font (size 1.27 1.27)) (justify left))
     )
@@
       (effects (font (size 1.27 1.27)) (justify left))
     )
-    (property "Value" "10k" (at 113.03 323.85 0)
+    (property "Value" "20k" (at 113.03 323.85 0)
       (effects (font (size 1.27 1.27)) (justify left))
     )
@@
       (effects (font (size 1.27 1.27)) (justify left))
     )
-    (property "Value" "10k" (at 147.32 323.85 0)
+    (property "Value" "20k" (at 147.32 323.85 0)
       (effects (font (size 1.27 1.27)) (justify left))
     )
@@
       (effects (font (size 1.27 1.27)) (justify left))
     )
-    (property "Value" "10k" (at 210.82 323.85 0)
+    (property "Value" "20k" (at 210.82 323.85 0)
       (effects (font (size 1.27 1.27)) (justify left))
     )
@@
       (effects (font (size 1.27 1.27)) (justify left))
     )
-    (property "Value" "10k" (at 185.42 323.85 0)
+    (property "Value" "20k" (at 185.42 323.85 0)
       (effects (font (size 1.27 1.27)) (justify left))
     )
@@
       (effects (font (size 1.27 1.27)) (justify left))
     )
-    (property "Value" "10k" (at 172.72 323.85 0)
+    (property "Value" "20k" (at 172.72 323.85 0)
       (effects (font (size 1.27 1.27)) (justify left))
     )
@@
       (effects (font (size 1.27 1.27)) (justify left))
     )
-    (property "Value" "10k" (at 236.22 323.85 0)
+    (property "Value" "20k" (at 236.22 323.85 0)
       (effects (font (size 1.27 1.27)) (justify left))
     )
